File: kicad/C64RAMCart.kicad_pcb (KiCad board)
At the start: 2 copper layers, 137 x 126.4 mm, 41 parts, among them J1 C64-Exp-Port_C64-Exp-Port, SW1 SW_SPST, SW2 SW_Push, SW3 SW_SPST, SW4 SW_Push, U1 2764, U10 KM62256CLP, U11 KM62256CLP, U2 74LS74, U3 6821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

Commit message: Gerbers and Schematic
Parts:
- removed ?: , 
- removed D4: LED_Small, LED_THT:LED_D5.0mm
- removed R4: R_Small, Resistor_THT:R_Axial_DIN0207_L6.3mm_D2.5mm_P7.62mm_Horizontal
- removed REF** (x4): 1pin, C64:M3_pin
- removed REF**: KiCad-Logo2_8mm_SilkScreen, Symbol:KiCad-Logo2_8mm_SilkScreen
- removed SW4: SW_Push, Button_Switch_THT:SW_PUSH_6mm_H7.3mm
- added H1: MountingHole, C64:M3_pin, F.Cu at (84.9, 40.1)
- added H2: MountingHole, C64:M3_pin, F.Cu at (212.2, 40.1)
- added H3: MountingHole, C64:M3_pin, F.Cu at (212.2, 127.1)
- added H4: MountingHole, C64:M3_pin, F.Cu at (84.4, 127.3)
Routing:
- net Net-(D4-Pad1): track 36.6 -> 0.00 mm
- net Net-(D4-Pad2): track 14.4 -> 0.00 mm

Commit message: RES fixed
Connections:
- SW2 pad 1: RES -> ~RES
- U2 pad 13: RES -> ~RES
- U3 pad 34: RES -> ~RES
- U4 pad 34: RES -> ~RES
Routing:
- net ~RES: track 0.00 -> 277.8 mm, vias 0 -> 1
- net RES: track 207.6 -> 0.00 mm, vias 1 -> 0
