File: kicad/C64RAMCart.sch (KiCad schematic (older format))
At the start: 16 parts, among them J1 C64-Exp-Port_C64-Exp-Port, SW2 SW_Push, SW3 SW_SPST, SW4 SW_Push, U1 2764, U2 74LS74, U3 6821, U4 6821, U5 74LS138

Commit message: Gerbers and Schematic
Parts:
- removed D4: LED_Small, LED_THT:LED_D5.0mm, symbol Device:LED_Small
- removed R4: R_Small, Resistor_THT:R_Axial_DIN0207_L6.3mm_D2.5mm_P7.62mm_Horizontal, symbol Device:R_Small
- removed SW4: SW_Push, Button_Switch_THT:SW_PUSH_6mm_H7.3mm, symbol Switch:SW_Push
Other:
- note removed: "RAM Battery Check"
Changed lines of the file:
@@
 encoding utf-8
 Sheet 1 2
-Title ""
-Date ""
-Rev ""
-Comp ""
-Comment1 ""
-Comment2 ""
-Comment3 ""
-Comment4 ""
+Title "Super Luxus CMOS RAM Platine"
+Date "2023-04-19"
+Rev "Rev001"
+Comp "Redrawn by AdamT117 (kayto@github.com)"
+Comment1 "designed and created by J Schucht."
+Comment2 "The design files are offered for educational purposes only."
+Comment3 "from the 64'er magazine dated March 1989"
+Comment4 "This C64 RAM cartridge is a recreation of the Super Luxus CMOS RAM Platine"
 $EndDescr
 $Comp
@@
 Text GLabel 9375 4425 0    50   Input ~ 0
 RES
-$Comp
-L Device:LED_Small D4
-U 1 1 63FD3B5C
-P 10575 4875
-F 0 "D4" V 10621 4805 50  0000 R CNN
-F 1 "LED_Small" V 10530 4805 50  0000 R CNN
-F 2 "LED_THT:LED_D5.0mm" V 10575 4875 50  0001 C CNN
-F 3 "~" V 10575 4875 50  0001 C CNN
-	1    10575 4875
-	0    -1   -1   0
-$EndComp
-$Comp
-L power:GND #PWR0112
-U 1 1 63FD464B
-P 10575 5475
-F 0 "#PWR0112" H 10575 5225 50  0001 C CNN
-F 1 "GND" H 10580 5302 50  0000 C CNN
-F 2 "" H 10575 5475 50  0001 C CNN
-F 3 "" H 10575 5475 50  0001 C CNN
-	1    10575 5475
-	1    0    0    -1
-$EndComp
-Wire Wire Line
-	10575 5050 10575 4975
-Wire Wire Line
-	10575 4775 10575 4700
-Wire Wire Line
-	10575 4175 10425 4175
-Text GLabel 10425 4175 0    50   Input ~ 0
-+5V
-$Comp
-L Device:R_Small R4
-U 1 1 640022A7
-P 10575 5150
-F 0 "R4" V 10771 5150 50  0000 C CNN
-F 1 "R_Small" V 10680 5150 50  0000 C CNN
-F 2 "Resistor_THT:R_Axial_DIN0207_L6.3mm_D2.5mm_P7.62mm_Horizontal" H 10575 5150 50  0001 C CNN
-F 3 "~" H 10575 5150 50  0001 C CNN
-	1    10575 5150
-	1    0    0    -1
-$EndComp
-Wire Wire Line
-	10575 5250 10575 5475
 Text Notes 9475 5850 0    50   ~ 0
 Reset
-Text Notes 10250 5850 0    50   ~ 0
-RAM Battery Check
-$Comp
-L Switch:SW_Push SW4
-U 1 1 63E472D1
-P 10575 4500
-F 0 "SW4" V 10529 4648 50  0000 L CNN
-F 1 "SW_Push" V 10620 4648 50  0000 L CNN
-F 2 "Button_Switch_THT:SW_PUSH_6mm_H7.3mm" H 10575 4700 50  0001 C CNN
-F 3 "~" H 10575 4700 50  0001 C CNN
-	1    10575 4500
-	0    1    1    0
-$EndComp
-Wire Wire Line
-	10575 4300 10575 4175
 Wire Bus Line
 	6250 4525 6250 5525

Commit message: RES fixed
Connections:
- net RES: no longer SW2.1, U3.34 (~RESET), U4.34 (~RESET)
- net ~RES: now also SW2.1, U3.34 (~RESET), U4.34 (~RESET)
Changed lines of the file:
@@
 	6375 3375 6125 3375
 Text GLabel 6125 3375 0    50   Input ~ 0
-RES
+~RES
 Wire Wire Line
 	6375 2775 6125 2775
@@
 	9350 3325 9100 3325
 Text GLabel 9100 3325 0    50   Input ~ 0
-RES
+~RES
 Wire Wire Line
 	9350 2725 9100 2725
@@
 	9575 4425 9375 4425
 Text GLabel 9375 4425 0    50   Input ~ 0
-RES
+~RES
 Text Notes 9475 5850 0    50   ~ 0
 Reset

Commit message: PCB and Schematic tidy
Parts:
- J1: value C64-Exp-Port_C64-Exp-Port -> C64-Exp-Port
- R2, R3: value R_Small -> 4k7
- RN1: value R_Network08 -> R_6k8_Network08
- RN2: value R_Network07 -> R_6k8_Network07
- renumbered C3 to 1nF1
Connections:
- net RES is gone; now on net ~RES: U2.13 (~R)
- net Vbb: now also R3.2, RN1.1 (common)
- net a13: no longer names the net of J1.J (A13)
- net a14: no longer names the net of J1.H (A14)
- net a15: no longer names the net of J1.F (A15)
- no-connect marks 23 -> 28
Other:
- note added: "E"
- moved on the sheet: 1nF1, J1, R2, R3, RN1, RN2, SW2, SW3, U1, U2A, U2B, U3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

Commit message: Remaining SRAM added
Parts:
- removed RN2: R_6k8_Network07, Resistor_THT:R_Array_SIP8, symbol Device:R_Network07
- added RN2: R_6k8_Network08, Resistor_THT:R_Array_SIP9, symbol Device:R_Network08
Connections:
- net Vcc: now also RN2.1 (common)
- net ar10: now also RN2.6 (R5)
- net ar11: now also RN2.5 (R4)
- net ar12: now also RN2.4 (R3)
- net ar13: now also RN2.3 (R2)
- net ar14: now also RN2.2 (R1)
- net ar8: now also RN2.8 (R7)
- net ar9: now also RN2.7 (R6)
- no-connect marks 28 -> 29
Changed lines of the file:
@@
 F1 "C64RAMCart_RAM.sch" 50
 $EndSheet
-$Comp
-L Device:R_Network07 RN2
-U 1 1 63EAEC02
-P 7625 3850
-F 0 "RN2" H 8025 3850 50  0000 L CNN
-F 1 "R_6k8_Network07" H 7475 4025 50  0000 L CNN
-F 2 "Resistor_THT:R_Array_SIP8" V 8100 3850 50  0001 C CNN
-F 3 "http://www.vishay.com/docs/31509/csc.pdf" H 7625 3850 50  0001 C CNN
-	1    7625 3850
-	-1   0    0    1
-$EndComp
 Entry Wire Line
 	8075 2275 7975 2375
@@
 Text GLabel 8600 6200 2    50   Output ~ 0
 Vbb
+$Comp
+L Device:R_Network08 RN2
+U 1 1 6448799E
+P 7525 3850
+AR Path="/6448799E" Ref="RN2"  Part="1"
+AR Path="/63E55187/6448799E" Ref="RN?"  Part="1"
+F 0 "RN2" H 7925 3850 50  0000 L CNN
+F 1 "R_6k8_Network08" H 7375 4025 50  0000 L CNN
+F 2 "Resistor_THT:R_Array_SIP9" V 8000 3850 50  0001 C CNN
+F 3 "http://www.vishay.com/docs/31509/csc.pdf" H 7525 3850 50  0001 C CNN
+	1    7525 3850
+	-1   0    0    1
+$EndComp
+NoConn ~ 7225 3650
 Wire Bus Line
 	5825 4525 5825 5525
